File: hardware/leds-hub/leds-hub.kicad_pcb (KiCad board)
At the start: 2 copper layers, 50 x 65 mm, 21 parts, among them J1 Conn_01x02, J10 Conn_01x02, J11 Conn_01x02, J12 Conn_01x02, J13 Conn_01x02, J14 Conn_01x02, J15 Conn_01x02, J16 Conn_01x02, J17 Conn_02x10_Odd_Even, J2 Conn_01x02, J3 Conn_01x02, J4 Conn_01x02, J5 Conn_01x02, J6 Conn_01x02, J7 Conn_01x02, J8 Conn_01x02, J9 Conn_01x02

Commit message: Refine PCB layout connections
Parts:
- moved J17 0.50 mm to (49.6, 131.5)
- renumbered J1 to LED01, J5 to LED02, J2 to LED03, J6 to LED04, J3 to LED05, J7 to LED06, J4 to LED07, J8 to LED08, J16 to LED09, J9 to LED10, J15 to LED11, J10 to LED12, J14 to LED13, J11 to LED14, J13 to LED15, J12 to LED16
Connections:
- net /+15V_LED renamed /V+_LED
- LED02 pad 2: /LED_05 -> /LED_02
- LED03 pad 2: /LED_02 -> /LED_03
- LED04 pad 2: /LED_06 -> /LED_04
- LED05 pad 2: /LED_03 -> /LED_05
- LED06 pad 2: /LED_07 -> /LED_06
- LED07 pad 2: /LED_04 -> /LED_07
- LED09 pad 2: /LED_16 -> /LED_09
- LED10 pad 2: /LED_09 -> /LED_10
- LED11 pad 2: /LED_15 -> /LED_11
- LED12 pad 2: /LED_10 -> /LED_12
- LED13 pad 2: /LED_14 -> /LED_13
- LED14 pad 2: /LED_11 -> /LED_14
- LED15 pad 2: /LED_13 -> /LED_15
- LED16 pad 2: /LED_12 -> /LED_16
Routing:
- net /LED_15: track 34.8 -> 61.2 mm
- net /LED_12: track 16.9 -> 38.4 mm
- net /LED_14: track 43.3 -> 27.1 mm
- net /LED_09: track 54.5 -> 39.3 mm
- net /LED_11: track 31.7 -> 46.6 mm
- net /LED_04: track 24.7 -> 38.8 mm
- net /LED_05: track 54.2 -> 42.0 mm
- net /LED_06: track 40.2 -> 28.2 mm
- net /LED_10: track 40.0 -> 50.7 mm
- net /LED_03: track 38.9 -> 49.4 mm
- net /LED_13: track 57.9 -> 53.9 mm
- net /LED_01: track 60.9 -> 57.1 mm
- net /LED_16: track 20.2 -> 16.7 mm
- net /LED_02: track 46.8 -> 49.3 mm
- net /LED_07: track 32.3 -> 34.7 mm
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Other:
- board text added: "16 LED CHANNELS HUB"
- board text added: "LED 1-16 V+ 17-20"
- board text removed: "16 LEDS HUB +15V - INDIVIDUAL CONTROL"
- board text removed: "LED 1-16 +15V 17-20"
