File: hardware/leds-hub/leds-hub.kicad_sch (KiCad schematic)
At the start: 17 parts, among them J1 Conn_01x02, J10 Conn_01x02, J11 Conn_01x02, J12 Conn_01x02, J13 Conn_01x02, J14 Conn_01x02, J15 Conn_01x02, J16 Conn_01x02, J17 Conn_02x10_Odd_Even, J2 Conn_01x02, J3 Conn_01x02, J4 Conn_01x02, J5 Conn_01x02, J6 Conn_01x02, J7 Conn_01x02, J8 Conn_01x02, J9 Conn_01x02

Commit message: Refine PCB layout connections
Parts:
- renumbered J1 to LED01, J2 to LED02, J3 to LED03, J4 to LED04, J5 to LED05, J6 to LED06, J7 to LED07, J8 to LED08, J9 to LED09, J10 to LED10, J11 to LED11, J12 to LED12, J13 to LED13, J14 to LED14, J15 to LED15, J16 to LED16
Connections:
- net +15V_LED renamed V+_LED
Other:
- moved on the sheet: J17
