File: hardware/controller/leds_controller/leds_controller.kicad_sch (KiCad schematic)
At the start: 5 parts, among them J1 Conn_02x10_Odd_Even, J2 XL6009_MODULE, U1 ULN2803A, U2 ULN2803A

Commit message: Work on PCB for the LED controller
Parts:
- A1: footprint Module:RaspberryPi_Pico_W_SMD_HandSolder -> Module:RaspberryPi_Pico_Common_Unspecified
- J2: footprint (none) -> Alpenhof:XL6009_Module_Socket
Connections:
- net CTRL_09: now also A1.21 (GPIO16); no longer A1.11 (GPIO8)
- net CTRL_10: now also A1.22 (GPIO17); no longer A1.12 (GPIO9)
- net CTRL_11: now also A1.24 (GPIO18); no longer A1.14 (GPIO10)
- net CTRL_12: now also A1.25 (GPIO19); no longer A1.15 (GPIO11)
- net CTRL_13: now also A1.26 (GPIO20); no longer A1.16 (GPIO12)
- net CTRL_14: now also A1.27 (GPIO21); no longer A1.17 (GPIO13)
- net CTRL_15: now also A1.29 (GPIO22); no longer A1.19 (GPIO14)
- net CTRL_16: now also A1.31 (GPIO26_ADC0); no longer A1.20 (GPIO15)
Changed lines of the file:
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@@
-	)
-	(no_connect
-		(at 73.66 71.12)
 	)
 	(no_connect
@@
 	)
 	(no_connect
-		(at 73.66 73.66)
+		(at 27.94 93.98)
 	)
 	(no_connect
-		(at 73.66 78.74)
+		(at 27.94 99.06)
 	)
 	(no_connect
-		(at 73.66 88.9)
+		(at 27.94 86.36)
 	)
 	(no_connect
-		(at 73.66 66.04)
+		(at 27.94 96.52)
+	)
+	(no_connect
+		(at 27.94 83.82)
+	)
+	(no_connect
+		(at 27.94 91.44)
 	)
 	(no_connect
@@
 	)
 	(no_connect
+		(at 27.94 81.28)
+	)
+	(no_connect
 		(at 27.94 53.34)
-	)
-	(no_connect
-		(at 73.66 63.5)
 	)
 	(no_connect
@@
 	)
 	(no_connect
-		(at 73.66 68.58)
-	)
-	(no_connect
-		(at 73.66 76.2)
+		(at 27.94 88.9)
 	)
 	(wire
@@
 	(wire
 		(pts
+			(xy 76.2 71.12) (xy 73.66 71.12)
+		)
+		(stroke
+			(width 0)
+			(type default)
+		)
+	)
+	(wire
+		(pts
 			(xy 125.73 48.26) (xy 123.19 48.26)
 		)
@@
 	(wire
 		(pts
-			(xy 25.4 88.9) (xy 27.94 88.9)
+			(xy 76.2 73.66) (xy 73.66 73.66)
 		)
 		(stroke
@@
 	(wire
 		(pts
+			(xy 76.2 63.5) (xy 73.66 63.5)
+		)
+		(stroke
+			(width 0)
+			(type default)
+		)
+	)
+	(wire
+		(pts
 			(xy 157.48 57.15) (xy 160.02 57.15)
 		)
@@
 	(wire
 		(pts
-			(xy 25.4 86.36) (xy 27.94 86.36)
-		)
-		(stroke
-			(width 0)
-			(type default)
-		)
-	)
-	(wire
-		(pts
 			(xy 157.48 72.39) (xy 160.02 72.39)
 		)
@@
 	(wire
 		(pts
+			(xy 76.2 76.2) (xy 73.66 76.2)
+		)
+		(stroke
+			(width 0)
+			(type default)
+		)
+	)
+	(wire
+		(pts
 			(xy 59.69 27.94) (xy 62.23 27.94)
 		)
@@
 	(wire
 		(pts
+			(xy 76.2 68.58) (xy 73.66 68.58)
+		)
+		(stroke
+			(width 0)
+			(type default)
+		)
+	)
+	(wire
+		(pts
 			(xy 175.26 74.93) (xy 172.72 74.93)
 		)
@@
 	(wire
 		(pts
-			(xy 25.4 96.52) (xy 27.94 96.52)
-		)
-		(stroke
-			(width 0)
-			(type default)
-		)
-	)
-	(wire
-		(pts
 			(xy 113.03 104.14) (xy 113.03 101.6)
 		)
@@
 	(wire
 		(pts
-			(xy 25.4 81.28) (xy 27.94 81.28)
-		)
-		(stroke
-			(width 0)
-			(type default)
-		)
-	)
-	(wire
-		(pts
 			(xy 175.26 77.47) (xy 172.72 77.47)
 		)
@@
 	(wire
 		(pts
-			(xy 25.4 83.82) (xy 27.94 83.82)
-		)
-		(stroke
-			(width 0)
-			(type default)
-		)
-	)
-	(wire
-		(pts
 			(xy 100.33 43.18) (xy 102.87 43.18)
 		)
@@
 	(wire
 		(pts
-			(xy 25.4 91.44) (xy 27.94 91.44)
-		)
-		(stroke
-			(width 0)
-			(type default)
-		)
-	)
-	(wire
-		(pts
 			(xy 125.73 35.56) (xy 123.19 35.56)
 		)
@@
 	(wire
 		(pts
+			(xy 76.2 66.04) (xy 73.66 66.04)
+		)
+		(stroke
+			(width 0)
+			(type default)
+		)
+	)
+	(wire
+		(pts
+			(xy 76.2 78.74) (xy 73.66 78.74)
+		)
+		(stroke
+			(width 0)
+			(type default)
+		)
+	)
+	(wire
+		(pts
 			(xy 125.73 86.36) (xy 123.19 86.36)
 		)
@@
 	(wire
 		(pts
-			(xy 25.4 99.06) (xy 27.94 99.06)
-		)
-		(stroke
-			(width 0)
-			(type default)
-		)
-	)
-	(wire
-		(pts
 			(xy 76.2 99.06) (xy 73.66 99.06)
 		)
@@
 	(wire
 		(pts
-			(xy 25.4 93.98) (xy 27.94 93.98)
-		)
-		(stroke
-			(width 0)
-			(type default)
-		)
-	)
-	(wire
-		(pts
 			(xy 125.73 45.72) (xy 123.19 45.72)
 		)
@@
 		(pts
 			(xy 100.33 45.72) (xy 102.87 45.72)
+		)
+		(stroke
+			(width 0)
+			(type default)
+		)
+	)
+	(wire
+		(pts
+			(xy 76.2 88.9) (xy 73.66 88.9)
 		)
 		(stroke
@@
 		)
 	)
-	(label "CTRL_14"
-		(at 25.4 93.98 180)
-		(effects
-			(font
-				(size 1.27 1.27)
-			)
-			(justify right bottom)
-		)
-	)
-	(label "CTRL_12"
-		(at 25.4 88.9 180)
-		(effects
-			(font
-				(size 1.27 1.27)
-			)
-			(justify right bottom)
-		)
-	)
 	(label "V+_LED"
 		(at 157.48 77.47 180)
@@
 		)
 	)
-	(label "CTRL_09"
-		(at 25.4 81.28 180)
-		(effects
-			(font
-				(size 1.27 1.27)
-			)
-			(justify right bottom)
+	(label "CTRL_13"
+		(at 76.2 73.66 0)
+		(effects
+			(font
+				(size 1.27 1.27)
+			)
+			(justify left bottom)
 		)
 	)
@@
 		)
 	)
+	(label "CTRL_12"
+		(at 76.2 71.12 0)
+		(effects
+			(font
+				(size 1.27 1.27)
+			)
+			(justify left bottom)
+		)
+	)
 	(label "CTRL_03"
 		(at 25.4 66.04 180)
@@
 		)
 	)
+	(label "CTRL_16"
+		(at 76.2 88.9 0)
+		(effects
+			(font
+				(size 1.27 1.27)
+			)
+			(justify left bottom)
+		)
+	)
 	(label "LED_08"
 		(at 175.26 62.23 0)
@@
 		)
 	)
+	(label "CTRL_10"
+		(at 76.2 66.04 0)
+		(effects
+			(font
+				(size 1.27 1.27)
+			)
+			(justify left bottom)
+		)
+	)
 	(label "CTRL_05"
 		(at 25.4 71.12 180)
@@
 		)
 	)
-	(label "CTRL_13"
-		(at 25.4 91.44 180)
-		(effects
-			(font
-				(size 1.27 1.27)
-			)
-			(justify right bottom)
-		)
-	)
 	(label "LED_10"
 		(at 175.26 64.77 0)
@@
 		)
 	)
+	(label "CTRL_14"
+		(at 76.2 76.2 0)
+		(effects
+			(font
+				(size 1.27 1.27)
+			)
+			(justify left bottom)
+		)
+	)
 	(label "CTRL_04"
 		(at 25.4 68.58 180)
@@
 		)
 	)
-	(label "CTRL_15"
-		(at 25.4 96.52 180)
-		(effects
-			(font
-				(size 1.27 1.27)
-			)
-			(justify right bottom)
-		)
-	)
 	(label "V+_LED"
 		(at 175.26 74.93 0)
@@
 		)
 	)
-	(label "CTRL_16"
-		(at 25.4 99.06 180)
-		(effects
-			(font
-				(size 1.27 1.27)
-			)
-			(justify right bottom)
-		)
-	)
 	(label "LED_04"
 		(at 175.26 57.15 0)
@@
 		)
 	)
+	(label "CTRL_15"
+		(at 76.2 78.74 0)
+		(effects
+			(font
+				(size 1.27 1.27)
+			)
+			(justify left bottom)
+		)
+	)
 	(label "LED_07"
 		(at 125.73 50.8 0)
@@
 		)
 	)
+	(label "CTRL_11"
+		(at 76.2 68.58 0)
+		(effects
+			(font
+				(size 1.27 1.27)
+			)
+			(justify left bottom)
+		)
+	)
 	(label "GND"
 		(at 76.2 99.06 0)
@@
 		)
 	)
+	(label "CTRL_09"
+		(at 76.2 63.5 0)
+		(effects
+			(font
+				(size 1.27 1.27)
+			)
+			(justify left bottom)
+		)
+	)
 	(label "LED_16"
 		(at 125.73 96.52 0)
@@
 		)
 	)
-	(label "CTRL_10"
-		(at 25.4 83.82 180)
-		(effects
-			(font
-				(size 1.27 1.27)
-			)
-			(justify right bottom)
-		)
-	)
 	(label "CTRL_05"
 		(at 100.33 45.72 180)
@@
 			)
 			(justify left bottom)
-		)
-	)
-	(label "CTRL_11"
-		(at 25.4 86.36 180)
-		(effects
-			(font
-				(size 1.27 1.27)
-			)
-			(justify right bottom)
 		)
 	)
@@
 			)
 		)
-		(property "Footprint" "Module:RaspberryPi_Pico_W_SMD_HandSolder"
+		(property "Footprint" "Module:RaspberryPi_Pico_Common_Unspecified"
 			(at 50.8 123.19 0)
 			(hide yes)
@@
 			)
 		)
-		(property "Footprint" ""
+		(property "Footprint" "Alpenhof:XL6009_Module_Socket"
 			(at 67.31 22.86 0)
 			(hide yes)
